File: powersection.kicad_sch (KiCad schematic)
At the start: 15 parts, among them IC3 BQ27441DRZR-G1A, IC4 TPS63001DRCR, J3 TSW-107-07-G-S

Commit message: feat: schematic v1
Parts:
- J3: footprint FP-TSW-107-07-G-S-MFG -> Connector_PinHeader_2.54mm:PinHeader_1x07_P2.54mm_Vertical
Other:
- note added: "BATT FUEL GAUGE"
- note added: "Buck-Boost Converter"
- note added: "PinHeader"
- moved on the sheet: C3, C4, C5, C6, C7, C8, IC3, IC4, J3, L1, R10, R11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
