File: projekt_Roland.kicad_sch (KiCad schematic)
At the start: 0 parts

Commit message: feat: schematic v1
Other:
- sheet  renamed USB-C
- added sheet BatteryCircuit (battery_circuit.kicad_sch)
- added sheet DC-DC Converter (untitled.kicad_sch)
- sheet USB-C: file Power section.kicad_sch -> usbc.kicad_sch
Changed lines of the file:
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@@
 	(generator_version "9.0")
 	(paper "A4")
+	(wire
+		(pts
+			(xy 91.44 71.12) (xy 102.87 71.12)
+		)
+		(stroke
+			(width 0)
+			(type default)
+		)
+	)
 	(sheet
-		(at 76.2 25.4)
-		(size 12.7 3.81)
+		(at 102.87 55.88)
+		(size 50.8 48.26)
+		(exclude_from_sim no)
+		(in_bom yes)
+		(on_board yes)
+		(dnp no)
+		(fields_autoplaced yes)
+		(stroke
+			(width 0.1524)
+			(type solid)
+		)
+		(fill
+			(color 0 0 0 0.0000)
+		)
+		(property "Sheetname" "DC-DC Converter"
+			(at 102.87 55.1684 0)
+			(effects
+				(font
+					(size 1.27 1.27)
+				)
+				(justify left bottom)
+			)
+		)
+		(property "Sheetfile" "untitled.kicad_sch"
+			(at 102.87 104.7246 0)
+			(effects
+				(font
+					(size 1.27 1.27)
+				)
+				(justify left top)
+			)
+		)
+		(pin "BAT+" input
+			(at 102.87 71.12 180)
+			(effects
+				(font
+					(size 1.27 1.27)
+				)
+				(justify left)
+			)
+		)
+		(instances
+			(project "projekt_Roland"
+				(path "/12081149-6dd0-47bb-bb21-fd1de250060f"
+					(page "5")
+				)
+			)
+		)
+	)
+	(sheet
+		(at 71.12 54.61)
+		(size 20.32 21.59)
 		(exclude_from_sim no)
 		(in_bom yes)
@@
 			(color 0 0 0 0.0000)
 		)
-		(property "Sheetname" ""
-			(at 76.2 24.6884 0)
+		(property "Sheetname" "BatteryCircuit"
+			(at 71.12 53.8984 0)
 			(effects
 				(font
@@
 			)
 		)
-		(property "Sheetfile" "powersection.kicad_sch"
-			(at 76.2 29.7946 0)
+		(property "Sheetfile" "battery_circuit.kicad_sch"
+			(at 71.12 76.7846 0)
 			(effects
 				(font
@@
 				)
 				(justify left top)
+			)
+		)
+		(pin "BAT_OUTPUT" output
+			(at 91.44 71.12 0)
+			(effects
+				(font
+					(size 1.27 1.27)
+				)
+				(justify right)
 			)
 		)
@@
 	)
 	(sheet
-		(at 25.4 25.4)
-		(size 12.7 3.81)
+		(at 71.12 83.82)
+		(size 17.78 21.59)
 		(exclude_from_sim no)
 		(in_bom yes)
@@
 			(color 0 0 0 0.0000)
 		)
-		(property "Sheetname" ""
-			(at 25.4 24.6884 0)
+		(property "Sheetname" "USB-C"
+			(at 71.12 83.1084 0)
 			(effects
 				(font
@@
 			)
 		)
-		(property "Sheetfile" "Power section.kicad_sch"
-			(at 25.4 29.7946 0)
+		(property "Sheetfile" "usbc.kicad_sch"
+			(at 71.12 105.9946 0)
 			(effects
 				(font
